File: NXP-Eagle-7.5.0/projects/NXPESC-UF1/NXPESC-UF1_test002.sch (EAGLE design)
At the start: 17 parts, among them J1 FLH1-03SZ-S3A-T, U1 MKV31F512VLL12-M, U2 PSMN1R4-30YLD, U3 PSMN1R4-30YLD, U4 PSMN1R4-30YLD, U5 PSMN1R4-30YLD, U6 PSMN1R4-30YLD, U7 PSMN1R4-30YLD

Commit message: Changing board name since i was locked out and saveed to NXP-Eagle-7.5.0/projects/NXPESC-UF1/NXPESC-UF1_test002.brd
Parts:
- removed J1: FLH1-03SZ-S3A-T, etc-connector-003a:FLH1-03SZ-S3A-T
- removed TP1: (no value), etc-connector-003a:TP-TH-SMLL
- removed U2, U3, U4, U5, U6, U7: PSMN1R4-30YLD, PSMN1R2-25YL_115:PSMN1R4-30YLD
- added C2, C3, C4, C5, C6, C7, C8, C9: CAP0603-150PF-50V, etc-rcl:CAP0603-150PF-50V
- added J2: FLH1-03SZ-S3A-T, etc-connector-003a:FLH1-03SZ-S3A-T
- added R10, R11, R12, R3, R8, R9: RESC0603-200R-1, etc-rcl:RESC0603-200R-1
- added R13, R14, R15, R16, R17, R18: RESC0603-1K-1, etc-rcl:RESC0603-1K-1
- added R19, R20, R21, R22, R23, R24, R25, R26: RESC0603-10K-1, etc-rcl:RESC0603-10K-1
- added TP2: (no value), etc-connector-003a:TP-TH-SMLL
- added U$3, U$4, U$5: FAN4852, NXPHLITE:FAN4852
- added U10, U11, U12, U13, U8, U9: PSMN1R4-30YLD, PSMN1R2-25YL_115:PSMN1R4-30YLD
- R1, R2, R4, R5: value RESC0603-200R-1 -> RESC2512-; device etc-rcl:RESC0603-200R-1 -> etc-rcl:RESC2512-
- R6, R7: value RESC0603-200R-1 -> RESC0603-1K-1; device etc-rcl:RESC0603-200R-1 -> etc-rcl:RESC0603-1K-1
Connections:
- removed net N$14: R5.2, U5.G
- new net +V_MOTOR: TP2.1, U10.D, U12.D, U8.D
- new net ADC_MID: C3.2, C5.2, C7.2, C9.2, R20.1, R22.1, R24.1, R26.1
- new net AGND: R16.1, R5.1
- new net CA_A_L: R14.2
- new net CS_ABC_L/DCB_H: R1.1, R14.1, R15.1, R18.1, R2.1, R4.1, R5.2, R7.1
- new net CS_A_H: C2.2, C6.2, C8.2, R13.2, R21.1, R23.1, R25.1, U$3.-IN1, U$4.-IN1, U$4.-IN2
- new net CS_A_L: C5.1, C7.1, C9.1, R22.2, R24.2, R26.2, U$3.+IN1, U$4.+IN1, U$4.+IN2
- new net CS_B_H: R17.2
- new net CS_B_L: R18.2
- new net CS_C_H: R6.2
- new net CS_C_L: R7.2
- new net CUR_DCB: C4.1, R19.2, U$5.OUT2
- new net N$1: R3.2, U8.G
- new net N$10: R11.2, U12.G
- new net N$17: R12.2, U13.G
- new net N$18: C2.1, R21.2, U$3.OUT1
- new net N$19: U$3.+VS
- new net N$20: U$4.+VS
- new net N$21: C6.1, R23.2, U$4.OUT1
- new net N$22: C8.1, R25.2, U$4.OUT2
- new net N$25: U$5.+VS
- new net N$3: R8.2, U9.G
- new net N$4: R9.2, U10.G
- new net N$9: R10.2, U11.G
- net GND: now also U$3.+IN2, U$3.-VS, U$4.-VS, U$5.-VS
- net HOA: now also R3.1; no longer R2.1
- net HOB: now also R9.1; no longer R4.1
- net HOC: now also R11.1; no longer R6.1
- net LOA: now also R8.1; no longer R1.1
- net LOB: now also R10.1; no longer R5.1
- net LOC: now also R12.1; no longer R7.1
- net N$11: now also R17.1, U11.S; no longer U2.G
- net N$12: now also R4.2, R6.1, U13.S; no longer R1.2, U3.G
- net N$13: now also U$3.-IN2, U$3.OUT2; no longer R4.2, U4.G
- net N$15: now also C3.1, R15.2, R20.2, U$5.+IN2; no longer R6.2, U6.G
- net N$16: now also C4.2, R16.2, R19.1, U$5.-IN2; no longer R7.2, U7.G
- net N$2: now also R1.2, R13.1, U9.S; no longer TP1.1, U2.D, U4.D, U6.D
- net PH_A: now also J2.1, U8.S, U9.D; no longer J1.1, U2.S, U3.D
- net PH_B: now also J2.2, U10.S, U11.D; no longer J1.2, U4.S, U5.D
- net PH_C: now also J2.3, U12.S, U13.D; no longer J1.3, U6.S, U7.D
Other:
- note added: "Value and wattage TBD Orginal was 0.02Ohm@1/2watt"
