File: NXP-Eagle-7.5.0/projects/NXPESC-UF1/NXPESC-UF1_test002.brd (EAGLE design)
At the start: 66 x 41.6 mm, 17 parts, among them J1 FLH1-03SZ-S3A-T, U1 MKV31F512VLL12-M, U2 PSMN1R4-30YLD, U3 PSMN1R4-30YLD, U4 PSMN1R4-30YLD, U5 PSMN1R4-30YLD, U6 PSMN1R4-30YLD, U7 PSMN1R4-30YLD

Commit message: Changing board name since i was locked out and saveed to NXP-Eagle-7.5.0/projects/NXPESC-UF1/NXPESC-UF1_test002.brd
Parts:
- removed J1: FLH1-03SZ-S3A-T, etc-connector-003a:J3
- removed TP1: (no value), etc-connector-003a:TP-SMLL
- removed U2, U3, U4, U5, U6, U7: PSMN1R4-30YLD, PSMN1R2-25YL_115:LFPAK56
- added C2, C3, C4, C5, C6, C7, C8, C9: CAP0603-150PF-50V, etc-rcl:C0603
- added J2: FLH1-03SZ-S3A-T, etc-connector-003a:J3
- added R10, R11, R12, R3, R8, R9: RESC0603-200R-1, etc-rcl:C0603
- added R13, R14, R15, R16, R17, R18: RESC0603-1K-1, etc-rcl:C0603
- added R19, R20, R21, R22, R23, R24, R25, R26: RESC0603-10K-1, etc-rcl:C0603
- added TP2: (no value), etc-connector-003a:TP-SMLL
- added U$3, U$4, U$5: FAN4852, NXPHLITE:SOP65P490X110-8N
- added U10, U11, U12, U13, U8, U9: PSMN1R4-30YLD, PSMN1R2-25YL_115:LFPAK56
- R1, R2, R4, R5: value RESC0603-200R-1 -> RESC2512-; device etc-rcl:C0603 -> etc-rcl:R2512
- R6, R7: value RESC0603-200R-1 -> RESC0603-1K-1
- moved R6 129.9 mm to (-7.37, -231.4)
- moved R7 129.9 mm to (-7.37, -236.5)
- moved R2 125.7 mm to (-5.08, -178.6)
- moved R1 113.2 mm to (-5.08, -171.2)
- moved R5 108.4 mm to (-5.08, -193.3)
- moved R4 106.1 mm to (-5.08, -185.9)
Connections:
- removed net N$14: R5.2, U5.4
- new net +V_MOTOR: TP2.1, U10.5, U12.5, U8.5
- new net ADC_MID: C3.2, C5.2, C7.2, C9.2, R20.1, R22.1, R24.1, R26.1
- new net AGND: R16.1, R5.1
- new net CA_A_L: R14.2
- new net CS_ABC_L/DCB_H: R1.1, R14.1, R15.1, R18.1, R2.1, R4.1, R5.2, R7.1
- new net CS_A_H: C2.2, C6.2, C8.2, R13.2, R21.1, R23.1, R25.1, U$3.2, U$4.2, U$4.6
- new net CS_A_L: C5.1, C7.1, C9.1, R22.2, R24.2, R26.2, U$3.3, U$4.3, U$4.5
- new net CS_B_H: R17.2
- new net CS_B_L: R18.2
- new net CS_C_H: R6.2
- new net CS_C_L: R7.2
- new net CUR_DCB: C4.1, R19.2, U$5.7
- new net N$1: R3.2, U8.4
- new net N$10: R11.2, U12.4
- new net N$17: R12.2, U13.4
- new net N$18: C2.1, R21.2, U$3.1
- new net N$19: U$3.8
- new net N$20: U$4.8
- new net N$21: C6.1, R23.2, U$4.1
- new net N$22: C8.1, R25.2, U$4.7
- new net N$25: U$5.8
- new net N$3: R8.2, U9.4
- new net N$4: R9.2, U10.4
- new net N$9: R10.2, U11.4
- net GND: now also U$3.4, U$3.5, U$4.4, U$5.4
- net HOA: now also R3.1; no longer R2.1
- net HOB: now also R9.1; no longer R4.1
- net HOC: now also R11.1; no longer R6.1
- net LOA: now also R8.1; no longer R1.1
- net LOB: now also R10.1; no longer R5.1
- net LOC: now also R12.1; no longer R7.1
- net N$11: now also R17.1, U11.1, U11.2, U11.3; no longer U2.4
- net N$12: now also R4.2, R6.1, U13.1, U13.2, U13.3; no longer R1.2, U3.4
- net N$13: now also U$3.6, U$3.7; no longer R4.2, U4.4
- net N$15: now also C3.1, R15.2, R20.2, U$5.5; no longer R6.2, U6.4
- net N$16: now also C4.2, R16.2, R19.1, U$5.6; no longer R7.2, U7.4
- net N$2: now also R1.2, R13.1, U9.1, U9.2, U9.3; no longer TP1.1, U2.5, U4.5, U6.5
- net PH_A: now also J2.1, U8.1, U8.2, U8.3, U9.5; no longer J1.1, U2.1, U2.2, U2.3, U3.5
- net PH_B: now also J2.2, U10.1, U10.2, U10.3, U11.5; no longer J1.2, U4.1, U4.2, U4.3, U5.5
- net PH_C: now also J2.3, U12.1, U12.2, U12.3, U13.5; no longer J1.3, U6.1, U6.2, U6.3, U7.5

Commit message: Adjusting board part placement too see how things are fitting. will need to compare with what other ESC layouts are like. Presently looking *quite* large!
Parts:
- moved C6 312.6 mm to (122.7, -54.1)
- moved C7 312.6 mm to (122.7, -59.2)
- moved C8 312.6 mm to (122.7, -74.4)
- moved C9 312.6 mm to (122.7, -79.5)
- moved R23 312.6 mm to (122.7, -64.3)
- moved R24 312.6 mm to (122.7, -69.3)
- moved R25 312.6 mm to (122.7, -84.6)
- moved R26 312.6 mm to (122.7, -89.7)
- moved U$4 312.6 mm to (125.2, -46.5)
- moved R15 312.3 mm to (122.7, -13.5)
- moved R17 312.3 mm to (122.7, 22.1)
- moved R22 312.3 mm to (122.7, -33.8)
- moved C2 312.3 mm to (122.7, -23.6)
- moved C3 312.3 mm to (122.7, -3.30)
- moved C4 312.3 mm to (122.7, -8.38)
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Routing:
- net VDD: track 29.7 -> 0.00 mm
- net N$7: track 18.6 -> 0.00 mm
- net N$6: track 11.4 -> 0.00 mm
Other:
- board size 66 x 41.6 mm -> 50.8 x 25.4 mm
